File: TS4231-BOB.kicad_sch (KiCad schematic)
At the start: 6 parts, among them J1 Conn_01x04, U1 TS4231

Commit message: update BOM
Parts:
- C1: Mfr # CL05B104KO5NNNC -> CC0603KRX7R7BB104
- C2: Mfr # CL05A105KP5NNNC -> CL10B105KO8NNNC
- R1: Mfr # ERJ-2RKF1502X -> ERJ-3EKF1502V
- U1: Mfr # (none) -> TS4231
Changed lines of the file:
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@@
 			)
 		)
-		(property "Datasheet" "https://media.digikey.com/pdf/Data%20Sheets/Samsung%20PDFs/CL05B104KO5NNNC.pdf"
+		(property "Datasheet" "https://www.yageo.com/upload/media/product/productsearch/datasheet/mlcc/UPY-GPHC_X7R_6.3V-to-250V_24.pdf"
 			(at 113.03 54.61 0)
 			(effects
@@
 			)
 		)
-		(property "Mfr #" "CL05B104KO5NNNC"
+		(property "Mfr #" "CC0603KRX7R7BB104"
 			(at 113.03 54.61 0)
 			(effects
@@
 			)
 		)
-		(property "Datasheet" "http://www.samsungsem.com/kr/support/product-search/mlcc/CL05A105KP5NNNC.jsp"
+		(property "Datasheet" "https://weblib.samsungsem.com/mlcc/mlcc-ec-data-sheet.do?partNumber=CL10B105KO8NNN"
 			(at 113.03 60.96 0)
 			(effects
@@
 			)
 		)
-		(property "Mfr #" "CL05A105KP5NNNC"
+		(property "Mfr #" "CL10B105KO8NNNC"
 			(at 113.03 60.96 0)
 			(effects
@@
 			)
 		)
-		(property "Mfr #" "ERJ-2RKF1502X"
+		(property "Mfr #" "ERJ-3EKF1502V"
 			(at 156.21 62.23 0)
 			(effects
@@
 			(at 139.7 49.53 0)
 			(effects
+				(font
+					(size 1.27 1.27)
+				)
+				(hide yes)
+			)
+		)
+		(property "Mfr #" "TS4231"
+			(at 139.7 49.53 0)
+			(effects
